File: board/eagle/projects/mimuz-ch55x/mimuz-ch55x.brd (EAGLE design)
At the start: 15 x 27 mm, 17 parts, among them P1 PINHEAD-1X7, P2 PINHEAD-1X7, P30 LED

Commit message: mod mimuz-ch55x.brd
Parts:
- moved U$1 0.05 mm to (7.50, 3.00)
Other:
- board text removed: "*"
- board text removed: "10K"
- board text removed: "CH552G"
- board text removed: "SW"
Changed lines of the file:
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@@
 <setting verticaltext="up"/>
 </settings>
-<grid distance="1" unitdist="mil" unit="mil" style="lines" multiple="1" display="yes" altdistance="5" altunitdist="mil" altunit="mil"/>
+<grid distance="0.5" unitdist="mm" unit="mm" style="lines" multiple="1" display="yes" altdistance="5" altunitdist="mil" altunit="mil"/>
 <layers>
 <layer number="1" name="Top" color="4" fill="1" visible="yes" active="yes"/>
 <layer number="2" name="Route2" color="16" fill="1" visible="no" active="no"/>
 <layer number="15" name="Route15" color="23" fill="1" visible="no" active="no"/>
-<layer number="16" name="Bottom" color="1" fill="1" visible="no" active="yes"/>
+<layer number="16" name="Bottom" color="1" fill="1" visible="yes" active="yes"/>
 <layer number="17" name="Pads" color="2" fill="1" visible="yes" active="yes"/>
 <layer number="18" name="Vias" color="2" fill="1" visible="yes" active="yes"/>
@@
 <layer number="20" name="Dimension" color="24" fill="1" visible="yes" active="yes"/>
 <layer number="21" name="tPlace" color="7" fill="1" visible="yes" active="yes"/>
-<layer number="22" name="bPlace" color="40" fill="1" visible="no" active="yes"/>
+<layer number="22" name="bPlace" color="40" fill="1" visible="yes" active="yes"/>
 <layer number="23" name="tOrigins" color="15" fill="1" visible="yes" active="yes"/>
 <layer number="24" name="bOrigins" color="15" fill="1" visible="yes" active="yes"/>
 <layer number="25" name="tNames" color="7" fill="1" visible="yes" active="yes"/>
-<layer number="26" name="bNames" color="40" fill="1" visible="no" active="yes"/>
+<layer number="26" name="bNames" color="40" fill="1" visible="yes" active="yes"/>
 <layer number="27" name="tValues" color="7" fill="1" visible="yes" active="yes"/>
-<layer number="28" name="bValues" color="40" fill="1" visible="no" active="yes"/>
+<layer number="28" name="bValues" color="40" fill="1" visible="yes" active="yes"/>
 <layer number="29" name="tStop" color="7" fill="3" visible="yes" active="yes"/>
 <layer number="30" name="bStop" color="7" fill="6" visible="yes" active="yes"/>
@@
 <text x="12.446" y="9.525" size="0.762" layer="22" font="vector" rot="SMR270" align="center">30</text>
 <text x="0.635" y="2.667" size="0.6096" layer="21" font="vector" rot="SR270" align="center">POW</text>
-<text x="4.7752" y="24.0284" size="0.6096" layer="21" font="vector" rot="SR0" align="center">10K</text>
-<text x="7.4168" y="25.2476" size="0.6096" layer="21" font="vector" rot="SR0" align="center">SW</text>
-<text x="7.4676" y="21.463" size="0.6096" layer="21" font="vector" rot="SR0" align="center">CH552G</text>
-<text x="8.8392" y="13.6652" size="1.27" layer="21" font="vector" rot="SR0" align="center">*</text>
 </plain>
 <attributes>
@@
 <element name="R1" library="0my" package="R0603" value="5.1K" x="10.6302" y="11.2" smashed="yes" rot="R270"/>
 <element name="R2" library="0my" package="R0603" value="5.1K" x="9.5" y="11.2" smashed="yes" rot="R270"/>
-<element name="*" library="ch552" package="SOIC16" value="CH552G" x="7.5" y="18.2" smashed="yes" rot="R90"/>
+<element name="*" library="ch552" package="SOIC16" value="CH552G" x="7.5" y="18.2" smashed="yes" rot="R90">
+<attribute name="NAME" x="9" y="13.985" size="0.6096" layer="25" font="vector" ratio="20" rot="R180" align="bottom-center"/>
+<attribute name="VALUE" x="7.5" y="22.55" size="0.6096" layer="27" font="vector" ratio="20" rot="R180" align="bottom-center"/>
+</element>
 <element name="U$2" library="ch552" package="USB-C" value="USB-C" x="7.5" y="6" smashed="yes"/>
 <element name="U$3" library="ch552" package="F1206" value="FUSE1206" x="8.5" y="8.6" smashed="yes" rot="R180"/>
-<element name="R3" library="0my" package="R0603" value="10K" x="3.4666" y="25.0334" smashed="yes" rot="R90"/>
+<element name="R3" library="0my" package="R0603" value="10K" x="3.4666" y="25.0334" smashed="yes" rot="R90">
+<attribute name="VALUE" x="3.91" y="23.2316" size="0.6096" layer="27" font="vector" align="center"/>
+</element>
 <element name="R4" library="0my" package="R0603" value="1K" x="13.5" y="6" smashed="yes" rot="R90"/>
 <element name="R5" library="0my" package="R0603" value="1.5K" x="1.5" y="6" smashed="yes" rot="R90"/>
-<element name="C1" library="0my" package="C0603" value="0.1u" x="5.135" y="10.274" smashed="yes" rot="R180"/>
-<element name="C2" library="0my" package="C0603" value="0.1u" x="4.7752" y="11.5904" smashed="yes"/>
-<element name="C3" library="0my" package="C0805" value="22u" x="4.254" y="8.3492" smashed="yes" rot="R180"/>
-<element name="U$1" library="logo" package="MIMUZ-SMALL" value="MIMUZ6MM" x="7.5" y="2.9464" smashed="yes" rot="MR0"/>
+<element name="C1" library="0my" package="C0603" value="0.1u" x="5.135" y="10.274" smashed="yes" rot="R180">
+<attribute name="VALUE" x="5.77" y="12.179" size="1.27" layer="27" rot="R180"/>
+</element>
+<element name="C2" library="0my" package="C0603" value="0.1u" x="4.7752" y="11.5904" smashed="yes">
+<attribute name="VALUE" x="4.1402" y="9.6854" size="1.27" layer="27"/>
+</element>
+<element name="C3" library="0my" package="C0805" value="22u" x="4.254" y="8.3492" smashed="yes" rot="R180">
+<attribute name="VALUE" x="5.524" y="10.8892" size="1.27" layer="27" rot="R180"/>
+</element>
+<element name="U$1" library="logo" package="MIMUZ-SMALL" value="MIMUZ6MM" x="7.5" y="3" smashed="yes" rot="MR0"/>
 <element name="POW" library="ch552" package="LED-0603" value="LED" x="1.651" y="2.794" smashed="yes" rot="R270"/>
 <element name="P30" library="ch552" package="LED-0603" value="LED" x="13.335" y="2.794" smashed="yes" rot="R270"/>
@@
 <vertex x="11.5" y="0" curve="-90"/>
 <vertex x="10.5" y="1"/>
-<vertex x="10.5" y="4" curve="90"/>
-<vertex x="8.5" y="6"/>
-<vertex x="6.5" y="6" curve="90"/>
-<vertex x="4.5" y="4"/>
+<vertex x="10.5" y="4.2" curve="90"/>
+<vertex x="8.5" y="6.2"/>
+<vertex x="6.5" y="6.2" curve="90"/>
+<vertex x="4.5" y="4.2"/>
 <vertex x="4.5" y="1" curve="-90"/>
 <vertex x="3.5" y="0"/>

Commit message: update board v1.0
Other:
- board text added: "2023/01/27 by @tadfmac"
- board text added: "ver.1.0"
- board text removed: "2023/01/21 by @tadfmac"
- board text removed: "ver.0.1"
Changed lines of the file:
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@@
 <grid distance="0.5" unitdist="mm" unit="mm" style="lines" multiple="1" display="yes" altdistance="5" altunitdist="mil" altunit="mil"/>
 <layers>
-<layer number="1" name="Top" color="4" fill="1" visible="yes" active="yes"/>
+<layer number="1" name="Top" color="4" fill="1" visible="no" active="yes"/>
 <layer number="2" name="Route2" color="16" fill="1" visible="no" active="no"/>
 <layer number="15" name="Route15" color="23" fill="1" visible="no" active="no"/>
-<layer number="16" name="Bottom" color="1" fill="1" visible="yes" active="yes"/>
+<layer number="16" name="Bottom" color="1" fill="1" visible="no" active="yes"/>
 <layer number="17" name="Pads" color="2" fill="1" visible="yes" active="yes"/>
 <layer number="18" name="Vias" color="2" fill="1" visible="yes" active="yes"/>
 <layer number="19" name="Unrouted" color="6" fill="1" visible="yes" active="yes"/>
 <layer number="20" name="Dimension" color="24" fill="1" visible="yes" active="yes"/>
-<layer number="21" name="tPlace" color="7" fill="1" visible="yes" active="yes"/>
+<layer number="21" name="tPlace" color="7" fill="1" visible="no" active="yes"/>
 <layer number="22" name="bPlace" color="40" fill="1" visible="yes" active="yes"/>
-<layer number="23" name="tOrigins" color="15" fill="1" visible="yes" active="yes"/>
+<layer number="23" name="tOrigins" color="15" fill="1" visible="no" active="yes"/>
 <layer number="24" name="bOrigins" color="15" fill="1" visible="yes" active="yes"/>
-<layer number="25" name="tNames" color="7" fill="1" visible="yes" active="yes"/>
+<layer number="25" name="tNames" color="7" fill="1" visible="no" active="yes"/>
 <layer number="26" name="bNames" color="40" fill="1" visible="yes" active="yes"/>
-<layer number="27" name="tValues" color="7" fill="1" visible="yes" active="yes"/>
+<layer number="27" name="tValues" color="7" fill="1" visible="no" active="yes"/>
 <layer number="28" name="bValues" color="40" fill="1" visible="yes" active="yes"/>
 <layer number="29" name="tStop" color="7" fill="3" visible="yes" active="yes"/>
@@
 <text x="0.6604" y="6.0198" size="0.6096" layer="21" font="vector" rot="SR270" align="center">1.5K</text>
 <text x="10" y="15.5" size="1.4224" layer="22" rot="MR270" align="center">mi:muz-ch55x</text>
-<text x="7.5" y="15.5" size="1.4224" layer="22" rot="MR270" align="center">ver.0.1</text>
-<text x="5" y="15.5" size="1.016" layer="22" rot="MR270" align="center">2023/01/21 by @tadfmac</text>
+<text x="7.5" y="15.5" size="1.4224" layer="22" rot="MR270" align="center">ver.1.0</text>
+<text x="5" y="15.5" size="1.016" layer="22" rot="MR270" align="center">2023/01/27 by @tadfmac</text>
 <text x="2.54" y="24.765" size="0.762" layer="22" font="vector" rot="MR270" align="center">11</text>
 <text x="2.54" y="22.225" size="0.762" layer="22" font="vector" rot="MR270" align="center">33</text>
@@
 <element name="R4" library="0my" package="R0603" value="1K" x="13.5" y="6" smashed="yes" rot="R90"/>
 <element name="R5" library="0my" package="R0603" value="1.5K" x="1.5" y="6" smashed="yes" rot="R90"/>
-<element name="C1" library="0my" package="C0603" value="0.1u" x="5.135" y="10.274" smashed="yes" rot="R180">
-<attribute name="VALUE" x="5.77" y="12.179" size="1.27" layer="27" rot="R180"/>
-</element>
-<element name="C2" library="0my" package="C0603" value="0.1u" x="4.7752" y="11.5904" smashed="yes">
-<attribute name="VALUE" x="4.1402" y="9.6854" size="1.27" layer="27"/>
-</element>
-<element name="C3" library="0my" package="C0805" value="22u" x="4.254" y="8.3492" smashed="yes" rot="R180">
-<attribute name="VALUE" x="5.524" y="10.8892" size="1.27" layer="27" rot="R180"/>
-</element>
+<element name="C1" library="0my" package="C0603" value="0.1u" x="5.135" y="10.274" smashed="yes" rot="R180"/>
+<element name="C2" library="0my" package="C0603" value="0.1u" x="4.7752" y="11.5904" smashed="yes"/>
+<element name="C3" library="0my" package="C0805" value="22u" x="4.254" y="8.3492" smashed="yes" rot="R180"/>
 <element name="U$1" library="logo" package="MIMUZ-SMALL" value="MIMUZ6MM" x="7.5" y="3" smashed="yes" rot="MR0"/>
 <element name="POW" library="ch552" package="LED-0603" value="LED" x="1.651" y="2.794" smashed="yes" rot="R270"/>
