File: board/eagle/projects/mimuz-ch55x/mimuz-ch55x.sch (EAGLE design)
At the start: 17 parts, among them P1 PINHEAD-1X7, P2 PINHEAD-1X7, P30 LED

Commit message: update board v1.0
Other:
- note added: "2023/01/27 by @tadfmac"
- note added: "mi:muz-ch55x v1.0"
- note removed: "2023/01/21 by @tadfmac"
- note removed: "mi:muz-ch55x v0.1"
Changed lines of the file:
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@@
 <sheet>
 <plain>
-<text x="55.88" y="152.4" size="7.62" layer="91" align="center">mi:muz-ch55x v0.1</text>
-<text x="55.88" y="144.78" size="2.54" layer="91" align="center">2023/01/21 by @tadfmac</text>
+<text x="55.88" y="152.4" size="7.62" layer="91" align="center">mi:muz-ch55x v1.0</text>
+<text x="55.88" y="144.78" size="2.54" layer="91" align="center">2023/01/27 by @tadfmac</text>
 </plain>
 <instances>
